File: Regulator.kicad_sch (KiCad schematic)
At the start: 12 parts, among them J1 1x4 Header, J2 1X4 Header, J3 1x4 Header

Commit message: Cleanup files and component linkage errors
Parts:
- F3: renamed from 3; footprint FP-0469-MFG -> AltiumImport:FP-0469-MFG
Changed lines of the file:
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@@
     (effects (font (size 1.27 1.27)) (justify left bottom))
   )
-  (label "5V Fuse" (at 165.1 104.14 0)
+  (label "5V Fuse" (at 165.1 104.14 0) (fields_autoplaced)
     (effects (font (size 1.27 1.27)) (justify left bottom))
   )
-  (label "12V Fuse" (at 119.38 86.36 0)
+  (label "12V Fuse" (at 119.38 86.36 0) (fields_autoplaced)
     (effects (font (size 1.27 1.27)) (justify left bottom))
   )
-  (label "Bat Fuse" (at 58.42 91.44 0)
+  (label "Bat Fuse" (at 58.42 91.44 0) (fields_autoplaced)
     (effects (font (size 1.27 1.27)) (justify left bottom))
   )
-  (label "Bat In" (at 25.4 83.82 0)
+  (label "Bat In" (at 25.4 83.82 0) (fields_autoplaced)
     (effects (font (size 1.27 1.27)) (justify left bottom))
   )
-  (label "Comp Out" (at 210.82 83.82 0)
+  (label "Comp Out" (at 210.82 83.82 0) (fields_autoplaced)
     (effects (font (size 1.27 1.27)) (justify left bottom))
   )
@@
   (symbol (lib_id "Regulator-altium-import:root_0_5bcf9b9f640e542cf0359d10258e979") (at 180.34 83.82 0) (unit 1)
     (in_bom yes) (on_board yes) (dnp no)
-    (property "Reference" "3" (at 184.404 79.756 0)
+    (property "Reference" "F3" (at 184.404 79.756 0)
       (effects (font (size 1.27 1.27)) (justify left bottom))
     )
@@
       (effects (font (size 1.27 1.27)) (justify left bottom) hide)
     )
-    (property "Footprint" "FP-0469-MFG" (at 180.34 83.82 0)
+    (property "Footprint" "AltiumImport:FP-0469-MFG" (at 180.34 83.82 0)
       (effects (font (size 1.27 1.27)) hide)
     )
@@
       (project "Regulator"
         (path "/eb9a600c-5129-4053-93d7-61ac26c94f1d"
-          (reference "3") (unit 1)
-        )
-      )
+          (reference "F3") (unit 1)
+        )
+      )

Commit message: Cleanup component properties and footprints table
Parts:
- D1, D2, D3: Part Number (none) -> SML-LX1206YC-TR
- F1: Part Number (none) -> 0466004.NR
- F2: Part Number (none) -> 0466003.NR
- F3: Part Number (none) -> 0466005.NR
- R1: footprint AltiumImport:FP-CR1206-IPC_B -> Resistor_SMD:R_1206_3216Metric_Pad1.30x1.75mm_HandSolder
- R2: footprint AltiumImport:FP-MCA1206-IPC_C -> Resistor_SMD:R_1206_3216Metric_Pad1.30x1.75mm_HandSolder
- R3: footprint AltiumImport:RESC3216X70X50LL05T20 -> Resistor_SMD:R_1206_3216Metric_Pad1.30x1.75mm_HandSolder
Changed lines of the file:
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@@
       (effects (font (size 1.27 1.27)) (justify left bottom) hide)
+    )
+    (property "Part Number" "SML-LX1206YC-TR" (at 60.96 109.22 0)
+      (effects (font (size 1.27 1.27)) hide)
     )
     (pin "1")
@@
       (effects (font (size 1.27 1.27)) (justify left bottom))
     )
-    (property "Footprint" "AltiumImport:FP-CR1206-IPC_B" (at 76.2 111.76 0)
+    (property "Footprint" "Resistor_SMD:R_1206_3216Metric_Pad1.30x1.75mm_HandSolder" (at 76.2 111.76 0)
       (effects (font (size 1.27 1.27)) hide)
     )
@@
       (effects (font (size 1.27 1.27)) (justify left bottom) hide)
     )
+    (property "Part Number" "" (at 76.2 111.76 0)
+      (effects (font (size 1.27 1.27)) hide)
+    )
     (pin "1")
     (pin "2")
@@
       (effects (font (size 1.27 1.27)) (justify left bottom) hide)
     )
+    (property "Part Number" "0466004.NR" (at 38.1 83.82 0)
+      (effects (font (size 1.27 1.27)) hide)
+    )
     (pin "1")
     (pin "2")
@@
       (effects (font (size 1.27 1.27)) (justify left bottom) hide)
     )
+    (property "Part Number" "SML-LX1206YC-TR" (at 203.2 99.06 0)
+      (effects (font (size 1.27 1.27)) hide)
+    )
     (pin "1")
     (pin "2")
@@
       (effects (font (size 1.27 1.27)) (justify left bottom))
     )
-    (property "Footprint" "AltiumImport:RESC3216X70X50LL05T20" (at 213.36 99.06 0)
+    (property "Footprint" "Resistor_SMD:R_1206_3216Metric_Pad1.30x1.75mm_HandSolder" (at 213.36 99.06 0)
       (effects (font (size 1.27 1.27)) hide)
     )
@@
       (effects (font (size 1.27 1.27)) (justify left bottom) hide)
     )
+    (property "Part Number" "" (at 213.36 99.06 0)
+      (effects (font (size 1.27 1.27)) hide)
+    )
     (pin "1")
     (pin "2")
@@
     (property "MANUFACTURER" "Littelfuse" (at 131.572 82.296 0)
       (effects (font (size 1.27 1.27)) (justify left bottom) hide)
+    )
+    (property "Part Number" "0466003.NR" (at 132.08 86.36 0)
+      (effects (font (size 1.27 1.27)) hide)
     )
     (pin "1")
@@
       (effects (font (size 1.27 1.27)) (justify left bottom) hide)
     )
+    (property "Part Number" "SML-LX1206YC-TR" (at 157.48 63.5 0)
+      (effects (font (size 1.27 1.27)) hide)
+    )
     (pin "1")
     (pin "2")
@@
       (effects (font (size 1.27 1.27)) (justify left bottom) hide)
     )
+    (property "Part Number" "0466005.NR" (at 180.34 83.82 0)
+      (effects (font (size 1.27 1.27)) hide)
+    )
     (pin "1")
     (pin "2")
@@
     (property "MANUFACTURER PART NUMBER" "61300411121" (at 101.6 83.82 0)
       (effects (font (size 1.27 1.27)) (justify left bottom) hide)
+    )
+    (property "Part Number" "" (at 111.76 81.28 0)
+      (effects (font (size 1.27 1.27)) hide)
     )
     (pin "1")
@@
       (effects (font (size 1.27 1.27)) (justify left bottom))
     )
-    (property "Footprint" "AltiumImport:FP-MCA1206-IPC_C" (at 165.1 66.04 0)
+    (property "Footprint" "Resistor_SMD:R_1206_3216Metric_Pad1.30x1.75mm_HandSolder" (at 165.1 66.04 0)
       (effects (font (size 1.27 1.27)) hide)
     )
@@
       (effects (font (size 1.27 1.27)) (justify left bottom) hide)
     )
+    (property "Part Number" "" (at 165.1 66.04 0)
+      (effects (font (size 1.27 1.27)) hide)
+    )
     (pin "1")
     (pin "2")
@@
     (property "MANUFACTURER PART NUMBER" "61300411121" (at 159.512 105.41 0)
       (effects (font (size 1.27 1.27)) (justify left bottom) hide)
+    )
+    (property "Part Number" "" (at 162.56 99.06 0)
+      (effects (font (size 1.27 1.27)) hide)
     )
     (pin "1")
@@
       (effects (font (size 1.27 1.27)) (justify left bottom) hide)
     )
-    (pin "1")
+    (property "Part Number" "" (at 83.82 99.06 0)
+      (effects (font (size 1.27 1.27)) hide)
+    )
+    (pin "1")

Commit message: Remove imported symbol table fiends
Parts:
- D1, D2, D3: CATALOG DRAWINGS SML-LX1206SeriesTopSML-LX1206SeriesSideSML-LX1206SeriesBott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 -> (none); CATEGORY Optoelectronics -> (none); COLOR Yellow -> (none); CURRENT - TEST 20mA -> (none); DATASHEET URL http://www.lumex.com/content/files/ProductAttachment/SML-LX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 -> (none); DATASHEET VERSION Rev. K, 08/2012 -> (none); FAMILY LEDIndication-Discrete -> (none); FEATURES - -> (none); HEIGHT (MAX) 1.10mm -> (none); LENS COLOR Colorless -> (none); LENS STYLE/SIZE RectanglewithFlatTop -> (none); LENS TRANSPARENCY Clear -> (none); MANUFACTURER Lumex -> (none); MANUFACTURER URL http://www.lumexinstruments.com/ -> (none); MILLICANDELA RATING 6mcd -> (none); MOUNTING TECHNOLOGY SurfaceMount -> (none); MOUNTING TYPE SurfaceMount -> (none); ONLINE CATALOG SML-LX1206RectanglewithFlatTop1206PackageLEDs -> (none); OTHER NAMES 67-1358-2LU60357TRSMLLX1206YCTR -> (none); PACKAGE / CASE 1206(3216Metric) -> (none); PACKAGE DESCRIPTION 2-Pin Surface Mount Device, Body 3.2 x 1.5 mm -> (none); PACKAGE REFERENCE SML-LX1206YC-TR -> (none); PACKAGING Tape&Reel(TR) -> (none); PRODUCT TRAINING MODULES LEDsBenefitsofCustomLEDandLCDTechnology -> (none); ROHS INFORMATION RoHSCertofCompliance -> (none); SERIES - -> (none); SIZE / DIMENSION 3.20mmLx1.60mmW -> (none); STANDARD PACKAGE 3,000 -> (none); SUPPLIER DEVICE PACKAGE 1206 -> (none); VIEWING ANGLE 160° -> (none); VOLTAGE - FORWARD (VF) (TYP) 2.1V -> (none); WAVELENGTH - DOMINANT - -> (none); WAVELENGTH - PEAK 585nm -> (none)
- F1: APPROVALS CE -> (none); CASE CODE (IMPERIAL) 1206 -> (none); CASE CODE (METRIC) 3216 -> (none); CASE/PACKAGE 1206 -> (none); CURRENT RATING 4A -> (none); DC COLD RESISTANCE 30mR -> (none); FUSE TYPE Board Mount (Cartridge Style Excluded) -> (none); MAX OPERATING TEMPERATURE 125°C -> (none); MIN OPERATING TEMPERATURE -55°C -> (none); MOUNT Surface Mount -> (none); PACKAGING Cut Tape -> (none); ROHS COMPLIANT Yes -> (none); VOLTAGE RATING (AC) 63V -> (none); VOLTAGE RATING (DC) 63V -> (none)
- F2: ALTIUM_VALUE 0.019Ω -> (none); AUTOMOTIVE No -> (none); CATEGORY Fuse -> (none); COMPONENTLINK2DESCRIPTION Datasheet -> (none); COMPONENTLINK2URL https://www.littelfuse.com/~/media/electronics/datasheets/f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 -> (none); DEVICE CLASS L1 Circuit Protection -> (none); DEVICE CLASS L2 Fuses -> (none); DEVICE CLASS L3 unset -> (none); DIGIKEY DESCRIPTION FUSE BOARD MNT 3A 32VAC/VDC 1206 -> (none); FUSE BLOW SPEED Fast -> (none); FUSE CURRENT 3A -> (none); FUSE I2T 0.576A2Sec -> (none); FUSE INTERRUPT AC CURRENT 50A -> (none); FUSE INTERRUPT DC CURRENT 50A -> (none); FUSE VOLTAGE DROP 75.99mV -> (none); HEIGHT 0.66mm -> (none); LEAD FREE Yes -> (none); MANUFACTURER Littelfuse -> (none); MANUFACTURER PART NUMBER 0466003.NR -> (none); MAX FUSE AC VOLTAGE 32V -> (none); MAX FUSE DC VOLTAGE 32V -> (none); MOUSER DESCRIPTION Surface Mount Fuses 32V 3A VFA Slimline -> (none); OCTOPART https://octopart.com/0466003.nr-littelfuse-565175 -> (none); PACKAGE 0466 -> (none); RESISTANCE 0.019Ω -> (none); ROHS TRUE -> (none); TEMPERATURE -55°C to +90°C -> (none); TEMPERATURE RANGE HIGH +90°C -> (none); TEMPERATURE RANGE LOW -55°C -> (none); VOLTAGE RATING 32V -> (none)
- F3: APPROVALS UL -> (none); BLOW CHARACTERISTIC TIME DELAY -> (none); BODY MATERIAL Ceramic -> (none); CASE CODE (IMPERIAL) 1206 -> (none); CASE CODE (METRIC) 3216 -> (none); CASE/PACKAGE 1206 -> (none); CURRENT RATING 5A -> (none); DC COLD RESISTANCE 35mR -> (none); DEPTH 1.63mm -> (none); FUSE CURRENT 5A -> (none); FUSE TYPE Board Mount (Cartridge Style Excluded) -> (none); HEIGHT 0.9mm -> (none); HOUSING MATERIAL Ceramic -> (none); LEAD FREE Lead Free -> (none); LENGTH 3.27mm -> (none); MAX OPERATING TEMPERATURE 150°C -> (none); MIN OPERATING TEMPERATURE -55°C -> (none); MOUNT Surface Mount -> (none); NUMBER OF PINS 2 -> (none); PACKAGE QUANTITY 3000 -> (none); PACKAGING Tape and Reel -> (none); POWER DISSIPATION 1.08W -> (none); RADIATION HARDENING No -> (none); RESISTANCE 35mR -> (none); RESISTOR TYPE Ceramic -> (none); ROHS COMPLIANT Yes -> (none); SERIES 469 -> (none); SIZE 0.9mm -> (none); TERMINAL MATERIAL Nickel -> (none); TERMINATION SMD/SMT -> (none); VOLTAGE RATING 32V -> (none); VOLTAGE RATING (DC) 32V -> (none); WIDTH 1.63mm -> (none); WORKING VOLTAGE 32V -> (none)
- J1, J2, J3: ALTIUM_VALUE 1x4 Header -> (none); MANUFACTURER Würth Elektronik -> (none); MANUFACTURER PART NUMBER 61300411121 -> (none)
- R1: CASE CODE (IMPERIAL) 1206 -> (none); CASE CODE (METRIC) 3216 -> (none); CASE/PACKAGE 1206 -> (none); COMPOSITION Thick Film -> (none); CONTACT PLATING Tin -> (none); DEPTH 1.6mm -> (none); FEATURES Moisture Resistant -> (none); HEIGHT 0.03inch -> (none); LENGTH 3.2mm -> (none); MAX OPERATING TEMPERATURE 155°C -> (none); MAX POWER DISSIPATION 250mW -> (none); MILITARY STANDARD Not -> (none); MIN OPERATING TEMPERATURE -55°C -> (none); MOUNT Surface Mount -> (none); NUMBER OF TERMINATIONS 2 -> (none); PACKAGE QUANTITY 5000 -> (none); PACKAGING Tape and Reel -> (none); POWER RATING 250mW -> (none); RADIATION HARDENING No -> (none); RESISTANCE 1.05kR -> (none); TEMPERATURE COEFFICIENT 100ppm/°C -> (none); TERMINATION SMD/SMT -> (none); THICKNESS 610um -> (none); TOLERANCE 1% -> (none); VOLTAGE RATING 200V -> (none); WIDTH 0.063inch -> (none)
- R2: CASE/PACKAGE 1206 -> (none); COMPOSITION Thin Film -> (none); HEIGHT 0.026inch -> (none); LEAD FREE Lead Free -> (none); LENGTH 0.126inch -> (none); MAX OPERATING TEMPERATURE 125°C -> (none); MAX POWER DISSIPATION 250mW -> (none); MIN OPERATING TEMPERATURE -55°C -> (none); NUMBER OF TERMINATIONS 2 -> (none); PACKAGE QUANTITY 5000 -> (none); PACKAGING Tape and Reel -> (none); RESISTANCE 800R -> (none); TEMPERATURE COEFFICIENT 25ppm/°C -> (none); TOLERANCE 0.1% -> (none); WIDTH 0.063inch -> (none)
- R3: MANUFACTURER Panasonic -> (none); PART NUMBER ERJ-8GEYJ201V -> (none)
